File: pcb/mosaic_usb/mosaic_usb.kicad_pcb (KiCad board)
At the start: 2 copper layers, 55 x 32 mm, 0 parts

Commit message: footprint and notes
Parts:
- added REF**: LED_D3.0mm_Clear_Sideways_Hack, 1_udu_lib:LED_D3.0mm_Clear_Sideways_Hack, F.Cu at (142.0, 78.0)
Changed lines of the file:
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@@
+		)
+	)
+	(footprint "1_udu_lib:LED_D3.0mm_Clear_Sideways_Hack"
+		(layer "F.Cu")
+		(at 142 78)
+		(descr "LED, diameter 3.0mm, 2 pins, clear, generated by kicad-footprint-generator")
+		(tags "LED")
+		(property "Reference" "REF**"
+			(at 1.27 -1.75 0)
+			(layer "F.SilkS")
+			(effects
+				(font
+					(size 1 1)
+					(thickness 0.15)
+				)
+			)
+		)
+		(property "Value" "LED_D3.0mm_Clear_Sideways_Hack"
+			(at 1.25 0 0)
+			(layer "F.Fab")
+			(effects
+				(font
+					(size 1 1)
+					(thickness 0.15)
+				)
+			)
+		)
+		(property "Datasheet" ""
+			(at 0 0 0)
+			(layer "F.Fab")
+			(hide yes)
+			(effects
+				(font
+					(size 1.27 1.27)
+				)
+			)
+		)
+		(property "Description" ""
+			(at 0 0 0)
+			(layer "F.Fab")
+			(hide yes)
+			(effects
+				(font
+					(size 1.27 1.27)
+				)
+			)
+		)
+		(property "KiLib_Generator" "LED/THT"
+			(at 0 0 0)
+			(layer "F.SilkS")
+			(hide yes)
+			(effects
+				(font
+					(size 1 1)
+					(thickness 0.15)
+				)
+			)
+		)
+		(attr through_hole)
+		(duplicate_pad_numbers_are_jumpers no)
+		(fp_line
+			(start -1.31 -1.16)
+			(end -1.022 -1.16)
+			(stroke
+				(width 0.12)
+				(type solid)
+			)
+			(layer "F.SilkS")
+		)
+		(fp_line
+			(start -1.16 -1.016)
+			(end -1.16 -1.304)
+			(stroke
+				(width 0.12)
+				(type solid)
+			)
+			(layer "F.SilkS")
+		)
+		(fp_line
+			(start -0.3 5)
+			(end -0.3 2.1)
+			(stroke
+				(width 0.1)
+				(type default)
+			)
+			(layer "Dwgs.User")
+		)
+		(fp_line
+			(start 0 1.3)
+			(end 0 -1.1)
+			(stroke
+				(width 0.1)
+				(type default)
+			)
+			(layer "Dwgs.User")
+		)
+		(fp_line
+			(start 2.6 1.3)
+			(end 2.6 -1.1)
+			(stroke
+				(width 0.1)
+				(type default)
+			)
+			(layer "Dwgs.User")
+		)
+		(fp_line
+			(start 2.82 5)
+			(end 2.82 2.08)
+			(stroke
+				(width 0.1)
+				(type default)
+			)
+			(layer "Dwgs.User")
+		)
+		(fp_rect
+			(start -0.7 1.29)
+			(end 3.2 2.08)
+			(stroke
+				(width 0.1)
+				(type default)
+			)
+			(fill no)
+			(layer "Dwgs.User")
+		)
+		(fp_arc
+			(start 2.82 5.03)
+			(mid 1.26 6.59)
+			(end -0.3 5.03)
+			(stroke
+				(width 0.1)
+				(type default)
+			)
+			(layer "Dwgs.User")
+		)
+		(fp_rect
+			(start -1.45 1.25)
+			(end 4.05 6.75)
+			(stroke
+				(width 0.1)
+				(type solid)
+			)
+			(fill no)
+			(layer "Cmts.User")
+		)
+		(fp_rect
+			(start -1.8 -1.5)
+			(end 4.4 7)
+			(stroke
+				(width 0.05)
+				(type solid)
+			)
+			(fill no)
+			(layer "F.CrtYd")
+		)
+		(fp_text user "${REFERENCE}"
+			(at 1.27 0 0)
+			(layer "F.Fab")
+			(effects
+				(font
+					(size 0.8 0.8)
+					(thickness 0.12)
+				)
+			)
+		)
+		(point
+			(at 143.27 78)
+			(size 2)
+			(layer "F.Fab")
+		)
+		(pad "1" smd rect
+			(at 0 0)
+			(size 1.8 1.8)
+			(layers "F.Cu" "F.Mask" "F.Paste")
+		)
+		(pad "2" smd circle
+			(at 2.54 0)
+			(size 1.8 1.8)
+			(layers "F.Cu" "F.Mask" "F.Paste")
+		)
+		(zone
+			(layer "F.Mask")
+			(hatch edge 0.5)
+			(connect_pads
+				(clearance 0)
+			)
+			(min_thickness 0.25)
+			(keepout
+				(tracks not_allowed)
+				(vias not_allowed)
+				(pads not_allowed)
+				(copperpour allowed)
+				(footprints allowed)
+			)
+			(placement
+				(enabled no)
+				(sheetname "")
+			)
+			(fill
+				(thermal_gap 0.5)
+				(thermal_bridge_width 0.5)
+				(island_removal_mode 0)
+			)
+			(polygon
+				(pts
+					(xy 140.6 79.3) (xy 146 79.3) (xy 146 84.7) (xy 140.6 84.7) (xy 140.6 78.9)
+				)
+			)
+		)
+		(embedded_fonts no)
+		(model "${KICAD10_3DMODEL_DIR}/LED_THT.3dshapes/LED_D3.0mm_Clear.step"
+			(offset
+				(xyz 0 1.5 2)
+			)
+			(scale
+				(xyz 1 1 1)
+			)
+			(rotate
+				(xyz -90 -0 -0)
+			)
 		)
 	)

Commit message: pcb layout
Parts:
- removed REF**: LED_D3.0mm_Clear_Sideways_Hack, 1_udu_lib:LED_D3.0mm_Clear_Sideways_Hack
- added BT1: CR2032, 1_udu_lib:BATT_HLDR_LNX, B.Cu at (111.7, 88.5)
- added D1: LED, 1_udu_lib:LED_D3.0mm_Clear_Sideways_Hack, B.Cu at (169.0, 29.5)
- added D10: LED, 1_udu_lib:LED_D3.0mm_Clear_Sideways_Hack, B.Cu at (120.0, 42.0)
- added D11: LED, 1_udu_lib:LED_D3.0mm_Clear_Sideways_Hack, B.Cu at (169.0, 53.1)
- added D12: LED, 1_udu_lib:LED_D3.0mm_Clear_Sideways_Hack, B.Cu at (156.0, 54.5)
- added D13: LED, 1_udu_lib:LED_D3.0mm_Clear_Sideways_Hack, B.Cu at (133.0, 89.1)
- added D14: LED, 1_udu_lib:LED_D3.0mm_Clear_Sideways_Hack, B.Cu at (131.2, 54.5)
- added D15: LED, 1_udu_lib:LED_D3.0mm_Clear_Sideways_Hack, B.Cu at (108.0, 30.1)
- added D16: LED, 1_udu_lib:LED_D3.0mm_Clear_Sideways_Hack, B.Cu at (169.0, 64.1)
- added D17: LED, 1_udu_lib:LED_D3.0mm_Clear_Sideways_Hack, B.Cu at (169.0, 89.1)
- added D18: LED, 1_udu_lib:LED_D3.0mm_Clear_Sideways_Hack, B.Cu at (144.0, 78.1)
- added D19: LED, 1_udu_lib:LED_D3.0mm_Clear_Sideways_Hack, B.Cu at (131.2, 67.1)
- added D2: LED, 1_udu_lib:LED_D3.0mm_Clear_Sideways_Hack, B.Cu at (156.0, 29.5)
- added D20: LED, 1_udu_lib:LED_D3.0mm_Clear_Sideways_Hack, B.Cu at (119.0, 67.1)
- added D3: LED, 1_udu_lib:LED_D3.0mm_Clear_Sideways_Hack, B.Cu at (143.4, 29.5)
- added D4: LED, 1_udu_lib:LED_D3.0mm_Clear_Sideways_Hack, B.Cu at (131.2, 29.5)
- added D5: LED, 1_udu_lib:LED_D3.0mm_Clear_Sideways_Hack, B.Cu at (108.0, 42.1)
- added D6: LED, 1_udu_lib:LED_D3.0mm_Clear_Sideways_Hack, B.Cu at (169.0, 42.0)
- added D7: LED, 1_udu_lib:LED_D3.0mm_Clear_Sideways_Hack, B.Cu at (157.0, 42.0)
- added D8: LED, 1_udu_lib:LED_D3.0mm_Clear_Sideways_Hack, B.Cu at (144.4, 42.0)
- added D9: LED, 1_udu_lib:LED_D3.0mm_Clear_Sideways_Hack, B.Cu at (132.2, 42.0)
- added J1: USB_A, PCM_Connector_USB_PCB_Edge:USB_A_PCB_Edge_receptacle, F.Cu at (88.0, 31.0)
- added R1: 330Ω, Resistor_SMD:R_0603_1608Metric, B.Cu at (66.2, 27.0)
- added R10: 330Ω, Resistor_SMD:R_0603_1608Metric, B.Cu at (62.2, 37.0)
- added R11: 330Ω, Resistor_SMD:R_0603_1608Metric, B.Cu at (58.2, 27.0)
- added R12: 330Ω, Resistor_SMD:R_0603_1608Metric, B.Cu at (58.2, 29.5)
- added R13: 330Ω, Resistor_SMD:R_0603_1608Metric, B.Cu at (58.2, 32.0)
- added R14: 330Ω, Resistor_SMD:R_0603_1608Metric, B.Cu at (58.2, 34.5)
- added R15: 330Ω, Resistor_SMD:R_0603_1608Metric, B.Cu at (58.2, 37.0)
- added R16: 330Ω, Resistor_SMD:R_0603_1608Metric, B.Cu at (54.2, 27.0)
- added R17: 330Ω, Resistor_SMD:R_0603_1608Metric, B.Cu at (54.2, 29.5)
- added R18: 330Ω, Resistor_SMD:R_0603_1608Metric, B.Cu at (54.2, 32.0)
- added R19: 330Ω, Resistor_SMD:R_0603_1608Metric, B.Cu at (54.2, 34.5)
- added R2: 330Ω, Resistor_SMD:R_0603_1608Metric, B.Cu at (66.2, 29.5)
- added R20: 330Ω, Resistor_SMD:R_0603_1608Metric, B.Cu at (54.2, 37.0)
- added R3: 330Ω, Resistor_SMD:R_0603_1608Metric, B.Cu at (66.2, 32.0)
- added R4: 330Ω, Resistor_SMD:R_0603_1608Metric, B.Cu at (66.2, 34.5)
- added R5: 330Ω, Resistor_SMD:R_0603_1608Metric, B.Cu at (66.2, 37.0)
- added R6: 330Ω, Resistor_SMD:R_0603_1608Metric, B.Cu at (62.2, 27.0)
- added R7: 330Ω, Resistor_SMD:R_0603_1608Metric, B.Cu at (62.2, 29.5)
- added R8: 330Ω, Resistor_SMD:R_0603_1608Metric, B.Cu at (62.2, 32.0)
- added R9: 330Ω, Resistor_SMD:R_0603_1608Metric, B.Cu at (62.2, 34.5)
Other:
- board size 55 x 32 mm -> 78 x 75 mm
- board text added: "PCB FAB Notes: 2.0mm Thickness"

Commit message: pcb footprint
Parts:
- added TP1: Mosaic Cube, 1_udu_lib:Mosaic Copper Cube, F.Cu at (118.0, 33.0)
- added TP2: Mosaic Cube, 1_udu_lib:Mosaic Copper Cube, F.Cu at (106.0, 57.0)
- added TP3: Mosaic Cube, 1_udu_lib:Mosaic Copper Cube, F.Cu at (130.0, 81.0)
- added TP5: Mosaic Cube, 1_udu_lib:Mosaic Copper Cube, F.Cu at (142.0, 58.0)
- added TP6: Mosaic Cube, 1_udu_lib:Mosaic Copper Cube, F.Cu at (144.0, 92.0)
- added TP7: Mosaic Cube, 1_udu_lib:Mosaic Copper Cube, F.Cu at (106.0, 93.0)
- added TP8: Mosaic Cube, 1_udu_lib:Mosaic Copper Cube, F.Cu at (156.0, 81.0)
- moved D3 38.8 mm to (117.2, 58.1)
- moved D14 27.2 mm to (154.2, 69.1)
- moved J1 5.00 mm to (93.0, 31.0)
- moved D10 4.44 mm to (118.2, 46.1)
- moved D16 4.29 mm to (167.0, 67.9)
- moved D20 4.02 mm to (118.0, 71.0)
- moved D9 3.66 mm to (129.2, 44.1)
- moved D1 3.61 mm to (167.0, 32.5)
- moved D13 3.61 mm to (131.0, 92.1)
- moved D17 3.61 mm to (167.0, 92.1)
- moved D18 3.61 mm to (142.0, 81.1)
- moved D4 3.61 mm to (129.2, 32.5)
- moved D5 3.61 mm to (106.0, 45.1)
- moved D6 3.61 mm to (167.0, 45.0)
- moved D7 3.61 mm to (155.0, 45.0)
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Other:
- outline, holes or cut-outs redrawn

Commit message: add pcb stand
Parts:
- added REF**: MouseBite-Part_2.0x4.5mm_inset_D0.5mm_P0.85mm_7h, Panelization:MouseBite-Part_2.0x4.5mm_inset_D0.5mm_P0.85mm_7h, F.Cu at (191.0, 76.0)
- added REF**: MouseBite-Part_2.0x4.5mm_inset_D0.5mm_P0.85mm_7h, Panelization:MouseBite-Part_2.0x4.5mm_inset_D0.5mm_P0.85mm_7h, F.Cu at (189.0, 49.0)
- added REF**: MouseBite-Part_2.0x4.5mm_inset_D0.5mm_P0.85mm_7h, Panelization:MouseBite-Part_2.0x4.5mm_inset_D0.5mm_P0.85mm_7h, F.Cu at (177.0, 42.0)
- added REF**: MouseBite-Part_2.0x4.5mm_inset_D0.5mm_P0.85mm_7h, Panelization:MouseBite-Part_2.0x4.5mm_inset_D0.5mm_P0.85mm_7h, F.Cu at (175.0, 42.0)
- added REF**: MouseBite-Part_2.0x4.5mm_inset_D0.5mm_P0.85mm_7h, Panelization:MouseBite-Part_2.0x4.5mm_inset_D0.5mm_P0.85mm_7h, F.Cu at (189.0, 76.0)
- added REF**: MouseBite-Part_2.0x4.5mm_inset_D0.5mm_P0.85mm_7h, Panelization:MouseBite-Part_2.0x4.5mm_inset_D0.5mm_P0.85mm_7h, F.Cu at (191.0, 49.0)
- added REF**: MouseBite-Part_2.0x4.5mm_inset_D0.5mm_P0.85mm_7h, Panelization:MouseBite-Part_2.0x4.5mm_inset_D0.5mm_P0.85mm_7h, F.Cu at (177.0, 83.0)
- added REF**: MouseBite-Part_2.0x4.5mm_inset_D0.5mm_P0.85mm_7h, Panelization:MouseBite-Part_2.0x4.5mm_inset_D0.5mm_P0.85mm_7h, F.Cu at (175.0, 83.0)
Routing:
- added copper zone on B.Cu, net (none)
- added copper zone on F.Cu, net (none)
Other:
- board size 78 x 75 mm -> 125 x 75 mm

Commit message: routing and placement
Parts:
- moved R17 128.7 mm to (169.7, 86.3), turned to 0 degrees
- moved R11 114.0 mm to (169.8, 50.4), turned to 0 degrees
- moved R16 111.9 mm to (161.1, 60.2), turned to -90 degrees
- moved R18 107.7 mm to (148.9, 83.3), turned to -90 degrees
- moved R12 105.7 mm to (160.9, 54.7), turned to -90 degrees
- moved R14 102.9 mm to (157.1, 63.0), turned to 0 degrees
- moved R6 101.4 mm to (162.9, 38.8), turned to 0 degrees
- moved R13 99.4 mm to (132.2, 98.3), turned to 0 degrees
- moved R1 95.6 mm to (161.8, 30.5), turned to 90 degrees
- moved R7 92.0 mm to (153.7, 39.0), turned to 0 degrees
- moved R2 83.7 mm to (150.0, 30.6), turned to 90 degrees
- moved R8 80.8 mm to (142.8, 38.5), turned to -90 degrees
- moved R19 75.7 mm to (123.9, 64.3), turned to 0 degrees
- moved R20 74.5 mm to (117.1, 77.1)
- moved R9 65.6 mm to (127.7, 38.8), turned to 0 degrees
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Routing:
- net GND: track 0.00 -> 444.0 mm, vias 0 -> 1
- net +3.3V: track 0.00 -> 299.0 mm, vias 0 -> 1
- net Net-(D16-A): track 0.00 -> 19.4 mm
- net Net-(D15-A): track 0.00 -> 17.0 mm
- net Net-(D6-A): track 0.00 -> 16.0 mm
- net Net-(D3-A): track 0.00 -> 9.82 mm
- net Net-(D14-A): track 0.00 -> 9.33 mm
- net Net-(D11-A): track 0.00 -> 9.30 mm
- net Net-(D18-A): track 0.00 -> 9.27 mm
- net Net-(D17-A): track 0.00 -> 9.13 mm
- net Net-(D20-A): track 0.00 -> 9.12 mm
- net Net-(D1-A): track 0.00 -> 9.09 mm
- net Net-(D2-A): track 0.00 -> 8.78 mm
- net Net-(D5-A): track 0.00 -> 8.64 mm
- net Net-(D19-A): track 0.00 -> 7.52 mm
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
Commit message: polish pcb
Parts:
- removed TP7, TP8: Mosaic Cube, 1_udu_lib:Mosaic Copper Cube
- added REF**: MountingHole_5mm, MountingHole:MountingHole_5mm, F.Cu at (176.0, 101.0)
- added TP4: Mosaic Cube, 1_udu_lib:Mosaic Copper Cube, F.Cu at (106.9, 93.5)
- moved TP5 26.9 mm to (156.7, 81.2)
Other:
- board size 125 x 75 mm -> 125 x 82 mm
- board text added: "designed by danny <3"
- board text added: "usb mosaic art"
