File: pcb/mosaic_usb/mosaic_usb.kicad_sch (KiCad schematic)
At the start: 0 parts

Commit message: footprint and notes
Parts:
- added BT1: CR2032, symbol Device:Battery
- added D1: LED, symbol Device:LED
- added J1: USB_A, symbol Connector:USB_A
- added R1: R, symbol Device:R
Connections:
- new net: D1.2 (A), R1.2
- new net +5V: BT1.1 (+), J1.1 (VBUS), R1.1
- new net GND: BT1.2 (-), D1.1 (K), J1.4 (GND), J1.SH (Shield)
- no-connect marks 0 -> 2

Commit message: pcb layout
Parts:
- added D10, D11, D12, D13, D14, D15, D16, D17, D18, D19, D2, D20, D3, D4, D5, D6, D7, D8, D9: LED, 1_udu_lib:LED_D3.0mm_Clear_Sideways_Hack, symbol Device:LED
- added R10, R11, R12, R13, R14, R15, R16, R17, R18, R19, R2, R20, R3, R4, R5, R6, R7, R8, R9: 330Ω, Resistor_SMD:R_0603_1608Metric, symbol Device:R
- BT1: footprint (none) -> 1_udu_lib:BATT_HLDR_LNX
- D1: footprint (none) -> 1_udu_lib:LED_D3.0mm_Clear_Sideways_Hack
- J1: footprint (none) -> PCM_Connector_USB_PCB_Edge:USB_A_PCB_Edge_receptacle
- R1: value R -> 330Ω; footprint (none) -> Resistor_SMD:R_0603_1608Metric
Connections:
- net GND: now also D10.1 (K), D11.1 (K), D12.1 (K), D13.1 (K), D14.1 (K), D15.1 (K), D16.1 (K), D17.1 (K), D18.1 (K), D19.1 (K), D2.1 (K), D20.1 (K), D3.1 (K), D4.1 (K), D5.1 (K), D6.1 (K), D7.1 (K), D8.1 (K), D9.1 (K)
- net +5V renamed +3.3V
- net +3.3V: now also R10.1, R11.1, R12.1, R13.1, R14.1, R15.1, R16.1, R17.1, R18.1, R19.1, R2.1, R20.1, R3.1, R4.1, R5.1, R6.1, R7.1, R8.1, R9.1
- new net: D17.2 (A), R17.2
- new net: D8.2 (A), R8.2
- new net: D4.2 (A), R4.2
- new net: D9.2 (A), R9.2
- new net: D2.2 (A), R2.2
- new net: D13.2 (A), R13.2
- new net: D20.2 (A), R20.2
- new net: D11.2 (A), R11.2
- new net: D16.2 (A), R16.2
- new net: D6.2 (A), R6.2
- new net: D12.2 (A), R12.2
- new net: D3.2 (A), R3.2
- new net: D19.2 (A), R19.2
- new net: D15.2 (A), R15.2
- new net: D7.2 (A), R7.2
- new net: D10.2 (A), R10.2
- new net: D18.2 (A), R18.2
- new net: D14.2 (A), R14.2
- new net: D5.2 (A), R5.2
Other:
- note added: "power delivery"
- note added: "this is to acknowledge the use of two voltages, just dont have the battery and usb in at the same time bruh"
- moved on the sheet: BT1, D1, J1, R1

Commit message: pcb footprint
Parts:
- added TP1, TP2, TP3, TP4, TP5, TP6, TP7, TP8: Mosaic Cube, 1_udu_lib:Mosaic Copper Cube, symbol Connector:TestPoint
Connections:
- no-connect marks 2 -> 10

Commit message: polish pcb
Parts:
- removed TP7, TP8: Mosaic Cube, 1_udu_lib:Mosaic Copper Cube, symbol Connector:TestPoint
Connections:
- no-connect marks 10 -> 8
Changed lines of the file:
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@@
 	(rectangle
 		(start 20.32 20.32)
-		(end 77.47 76.2)
+		(end 76.2 76.2)
 		(stroke
 			(width 0)
@@
 	)
 	(no_connect
-		(at 31.75 132.08)
-	)
-	(no_connect
 		(at 31.75 93.98)
 	)
@@
 	)
 	(no_connect
-		(at 31.75 138.43)
-	)
-	(no_connect
 		(at 31.75 125.73)
 	)
@@
 	)
 	(symbol
-		(lib_id "Connector:TestPoint")
-		(at 31.75 132.08 0)
-		(unit 1)
-		(body_style 1)
-		(exclude_from_sim no)
-		(in_bom yes)
-		(on_board yes)
-		(in_pos_files yes)
-		(dnp no)
-		(fields_autoplaced yes)
-		(property "Reference" "TP7"
-			(at 34.29 127.5079 0)
-			(show_name no)
-			(do_not_autoplace no)
-			(effects
-				(font
-					(size 1.27 1.27)
-				)
-				(justify left)
-			)
-		)
-		(property "Value" "Mosaic Cube"
-			(at 34.29 130.0479 0)
-			(show_name no)
-			(do_not_autoplace no)
-			(effects
-				(font
-					(size 1.27 1.27)
-				)
-				(justify left)
-			)
-		)
-		(property "Footprint" "1_udu_lib:Mosaic Copper Cube"
-			(at 36.83 132.08 0)
-			(hide yes)
-			(show_name no)
-			(do_not_autoplace no)
-			(effects
-				(font
-					(size 1.27 1.27)
-				)
-			)
-		)
-		(property "Datasheet" ""
-			(at 36.83 132.08 0)
-			(hide yes)
-			(show_name no)
-			(do_not_autoplace no)
-			(effects
-				(font
-					(size 1.27 1.27)
-				)
-			)
-		)
-		(property "Description" "test point"
-			(at 31.75 132.08 0)
-			(hide yes)
-			(show_name no)
-			(do_not_autoplace no)
-			(effects
-				(font
-					(size 1.27 1.27)
-				)
-			)
-		)
-		(pin "1"
-		)
-		(instances
-			(project "mosaic_usb"
-				(path "/39b6eca2-17a5-4f4a-9003-524e14d0003d"
-					(reference "TP7")
-					(unit 1)
-				)
-			)
-		)
-	)
-	(symbol
 		(lib_id "Device:R")
 		(at 190.5 86.36 90)
@@
 					(unit 1)
 				)
-			)
-		)
-	)
-	(symbol
-		(lib_id "Connector:TestPoint")
-		(at 31.75 138.43 0)
-		(unit 1)
-		(body_style 1)
-		(exclude_from_sim no)
-		(in_bom yes)
-		(on_board yes)
-		(in_pos_files yes)
-		(dnp no)
-		(fields_autoplaced yes)
-		(property "Reference" "TP8"
-			(at 34.29 133.8579 0)
-			(show_name no)
-			(do_not_autoplace no)
-			(effects
-				(font
-					(size 1.27 1.27)
-				)
-				(justify left)
-			)
-		)
-		(property "Value" "Mosaic Cube"
-			(at 34.29 136.3979 0)
-			(show_name no)
-			(do_not_autoplace no)
-			(effects
-				(font
-					(size 1.27 1.27)
-				)
-				(justify left)
-			)
-		)
-		(property "Footprint" "1_udu_lib:Mosaic Copper Cube"
-			(at 36.83 138.43 0)
-			(hide yes)
-			(show_name no)
-			(do_not_autoplace no)
-			(effects
-				(font
-					(size 1.27 1.27)
-				)
-			)
-		)
-		(property "Datasheet" ""
-			(at 36.83 138.43 0)
-			(hide yes)
-			(show_name no)
-			(do_not_autoplace no)
-			(effects
-				(font
-					(size 1.27 1.27)
-				)
-			)
-		)
-		(property "Description" "test point"
-			(at 31.75 138.43 0)
-			(hide yes)
-			(show_name no)
-			(do_not_autoplace no)
-			(effects
-				(font
-					(size 1.27 1.27)
-				)
-			)
-		)
-		(pin "1"
-		)
-		(instances
-			(project "mosaic_usb"
-				(path "/39b6eca2-17a5-4f4a-9003-524e14d0003d"
-					(reference "TP8")
-					(unit 1)
-				)
